File: sang.sch (EAGLE design)
At the start: 27 parts, among them IC1 L293D, IC2 L293D, IC3 NE555, Q1 16MHz

Commit message: Pins BrokenOut - Pullups Changed
Internal Pull ups to be used, aded I2C pullups
Broke ut unused pin
Parts:
- added 12VOUT, 5VOUT: (no value), pinhead:PINHD-1X2
- added JP2: (no value), adafruit:PINHD-1X8BIG
- added R5: (no value), resistor:R-EU_0204/7
- R3: value 10K -> (none); device resistor:R-EU_0207/10 -> resistor:R-EU_0204/7
Connections:
- new net N$15: JP2.8, U$1.(PCINT8/T0/XCK)PB0
- new net N$16: JP2.7, U$1.(PCINT9/T1/CLKO)PB1
- new net N$17: JP2.6, U$1.(PCINT10/AIN0/INT2)PB2
- new net N$18: JP2.5, U$1.(PCINT11/AIN1/OC0A)PB3
- new net N$19: JP2.4, U$1.(PCINT12/OC0B/SS)PB4
- net +12V: now also 12VOUT.1, R1.2
- net +24V: now also R1.1
- net +5V: now also 5VOUT.1, R3.2, R5.2; no longer R1.2, START.3, START.4
- net GND: now also 12VOUT.2, 5VOUT.2, START.3, START.4; no longer R3.1
- net GO: no longer R3.2
- net MISO: now also JP2.2
- net MOSI: now also JP2.3
- net RST: no longer R1.1
- net SCK: now also JP2.1
- net SCL: now also R5.1
- net SDA: now also R3.1
Other:
- moved on the sheet: JP1, R1, R3
